File: ZX Dandanator Mini 2.1b.kicad_sch (KiCad schematic)
At the start: 28 parts, among them J1 ZX_48K_EDGE, J2 ZX_48K_EDGE, J3 Conn_01x06, J4 Conn_01x05, SW1 SW_PUSH, SW2 SW_PUSH, U1 PIC16F1826, U2 GAL22V10, U3 SST 39SF040

Commit message: small fix
Parts:
- C1, C2, C3, C4, C5: value 100nf -> 100nF
- D1, D2: value 1n4148 -> 1N4148
Other:
- note added: "* NOTE: Install C3 only in bare ZX Dandanator. If use Multiply (i.e. de arduino and sd card slot) do not install"
- moved on the sheet: A1, C1, C2, C3, C4, C5, D1, D2, DB1, H1, H2, H3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
