File: ZX Dandanator Mini 2.1b.kicad_pcb (KiCad board)
At the start: 2 copper layers, 88.9 x 79.6 mm, 28 parts, among them J1 ZX_48K_EDGE, J2 ZX_48K_EDGE, J3 Conn_01x06, J4 Conn_01x05, SW1 SW_PUSH, SW2 SW_PUSH, U1 PIC16F1826, U2 GAL22V10, U3 SST 39SF040

Commit message: retoques
Routing:
- net GND: track 328.5 -> 337.9 mm
- net RFSH: track 72.8 -> 76.4 mm
- net Mul-RX: track 74.4 -> 76.1 mm
- net A0: track 89.5 -> 90.8 mm
- net A2: track 85.7 -> 84.7 mm
- net HALT: track 75.4 -> 76.3 mm
- net PT_ROMCS: track 71.8 -> 72.7 mm
- net WR: track 122.4 -> 121.6 mm
- net NMI: track 121.7 -> 121.1 mm
- net V: track 78.2 -> 78.7 mm

Commit message: logos
Parts:
- added REF**: OSHW-Logo2_7.3x6mm_SilkScreen, Symbol:OSHW-Logo2_7.3x6mm_SilkScreen, F.Cu at (136.2, 60.0)
- added REF**: KiCad-Logo2_5mm_SilkScreen, Symbol:KiCad-Logo2_5mm_SilkScreen, F.Cu at (136.0, 71.1)
- moved J3 0.51 mm to (161.5, 61.4)
- moved H6 0.49 mm to (198.1, 57.8)
- moved H5 0.48 mm to (160.2, 57.8)
- moved H4 0.33 mm to (198.1, 77.7)
- moved H3 0.32 mm to (160.2, 77.7)
Routing:
- net GND: track 337.9 -> 340.1 mm
- net MOSI: track 37.5 -> 36.2 mm
- net SCK: track 54.8 -> 53.6 mm
- net MISO: track 37.5 -> 36.2 mm
- net Net-(A1-Pad27): track 106.5 -> 107.6 mm
- net CS: track 38.5 -> 37.9 mm
